Commit message: Update sim_house.sdf.xacro

File: tb_worlds/worlds/sim_house.sdf.xacro (robot description, xacro)
@@ -1,243 +1,1683 @@
-<?xml version='1.0' encoding='ASCII'?>
-<sdf version='1.7'>
-  <world name='warehouse'>
-    <physics type="ode">
-      <max_step_size>0.003</max_step_size>
-      <real_time_factor>1.0</real_time_factor>
-    </physics>
-    <plugin name="gz::sim::systems::Physics" filename="gz-sim-physics-system" />
-    <plugin name="gz::sim::systems::UserCommands" filename="gz-sim-user-commands-system" />
-    <plugin name="gz::sim::systems::SceneBroadcaster" filename="gz-sim-scene-broadcaster-system" />
-    <plugin name="gz::sim::systems::Contact" filename="gz-sim-contact-system" />
-    <!--<plugin name="gz::sim::systems::Sensors" filename="gz-sim-sensors-system">
-        <render_engine>ogre2</render_engine>
-    </plugin>-->
-    <scene>
-      <ambient>1 1 1 1</ambient>
-      <background>0.3 0.7 0.9 1</background>
-      <shadows>0</shadows>
-      <grid>false</grid>
-    </scene>
-    <!-- TODO(rkreinin): Fix lighting so that spawning multiple robots does not crash the sim-->
-    <!-- <light type="directional" name="sun">
+<?xml version="1.0"?>
+<sdf version="1.6" xmlns:xacro="http://www.ros.org/wiki/xacro">
+  <xacro:arg name="headless" default="false"/>
+  <world name='default'>
+    <plugin
+      filename="gz-sim-physics-system"
+      name="gz::sim::systems::Physics">
+    </plugin>
+    <plugin
+      filename="gz-sim-user-commands-system"
+      name="gz::sim::systems::UserCommands">
+    </plugin>
+    <plugin
+      filename="gz-sim-navsat-system"
+      name="gz::sim::systems::NavSat">
+    </plugin>
+  <xacro:unless value="$(arg headless)">
+    <plugin
+      filename="gz-sim-scene-broadcaster-system"
+      name="gz::sim::systems::SceneBroadcaster">
+    </plugin>
+  </xacro:unless>
+    <plugin
+      filename="gz-sim-sensors-system"
+      name="gz::sim::systems::Sensors">
+      <render_engine>ogre2</render_engine>
+    </plugin>
+    <plugin
+      filename="gz-sim-imu-system"
+      name="gz::sim::systems::Imu">
+    </plugin>
+    <light name='sun' type='directional'>
       <cast_shadows>0</cast_shadows>
-      <pose>-5 -3 10 0 0 0</pose>
-      <diffuse>1 1 1 1</diffuse>
-      <specular>1 1 1 1</specular>
-      <direction>0 0 -1</direction>
-    </light> -->
+      <pose>0 0 10 0 -0 0</pose>
+      <diffuse>0.8 0.8 0.8 1</diffuse>
+      <specular>0.2 0.2 0.2 1</specular>
+      <attenuation>
+        <range>1000</range>
+        <constant>0.9</constant>
+        <linear>0.01</linear>
+        <quadratic>0.001</quadratic>
+      </attenuation>
+      <direction>-0.5 0.1 -0.9</direction>
+      <spot>
+        <inner_angle>0</inner_angle>
+        <outer_angle>0</outer_angle>
+        <falloff>0</falloff>
+      </spot>
+    </light>
     <model name='ground_plane'>
-      <static>true</static>
+      <static>1</static>
       <link name='link'>
         <collision name='collision'>
           <geometry>
             <plane>
-              <normal>0.0 0.0 1</normal>
-              <size>1 1</size>
+              <normal>0 0 1</normal>
+              <size>100 100</size>
             </plane>
           </geometry>
-        </collision>
-      </link>
-      <pose>0 0 0 0 0 0</pose>
+          <surface>
+            <contact>
+              <collide_bitmask>65535</collide_bitmask>
+              <ode/>
+            </contact>
+            <friction>
+              <ode>
+                <mu>100</mu>
+                <mu2>50</mu2>
+              </ode>
+              <torsional>
+                <ode/>
+              </torsional>
+            </friction>
+            <bounce/>
+          </surface>
+          <max_contacts>10</max_contacts>
+        </collision>
+        <visual name='visual'>
+          <cast_shadows>0</cast_shadows>
+          <geometry>
+            <plane>
+              <normal>0 0 1</normal>
+              <size>100 100</size>
+            </plane>
+          </geometry>
+          <material>
+            <script>
+              <uri>file://media/materials/scripts/gazebo.material</uri>
+              <name>Gazebo/Grey</name>
+            </script>
+          </material>
+        </visual>
+        <self_collide>0</self_collide>
+        <enable_wind>0</enable_wind>
+        <kinematic>0</kinematic>
+      </link>
     </model>
-    <!-- Base -->
-    <include>
-      <uri>
-        https://fuel.gazebosim.org/1.0/OpenRobotics/models/Warehouse
-      </uri>
-      <name>warehouse</name>
-      <pose>0 0 -0.1 0 0 0</pose>
-    </include>
-    <!-- Pallet Box Mobile -->
-    <!--
-    <include>
-      <uri>
-        https://fuel.gazebosim.org/1.0/MovAi/models/pallet_box_mobile
-      </uri>
-      <name>pallet_box_0</name>
-      <pose>-4 12 0.01 0 0 0</pose>
-      <static>true</static>
-    </include> -->
-    <!-- Shelves -->
-    <include>
-      <uri>
-        https://fuel.gazebosim.org/1.0/MovAi/models/shelf_big
-      </uri>
-      <name>shelf_big_0</name>
-      <pose>-8.5 -13 0 0 -0 0</pose>
-    </include>
-    <include>
-      <uri>
-        https://fuel.gazebosim.org/1.0/MovAi/models/shelf_big
-      </uri>
-      <name>shelf_big_1</name>
-      <pose>6.5 -13 0 0 -0 0</pose>
-    </include>
-    <include>
-      <uri>
-        https://fuel.gazebosim.org/1.0/MovAi/models/shelf_big
-      </uri>
-      <name>shelf_big_2</name>
-      <pose>-1.5 -13 0 0 -0 0</pose>
-    </include>
-    <include>
-      <uri>
-        https://fuel.gazebosim.org/1.0/MovAi/models/shelf
-      </uri>
-      <name>shelf_3</name>
-      <pose>13.5 4.5 0 0 -0 0</pose>
-    </include>
-    <include>
-      <uri>
-        https://fuel.gazebosim.org/1.0/MovAi/models/shelf
-      </uri>
-      <name>shelf_4</name>
-      <pose>10 4.5 0 0 -0 0</pose>
-    </include>
-    <include>
-      <uri>
-        https://fuel.gazebosim.org/1.0/MovAi/models/shelf
-      </uri>
-      <name>shelf_5</name>
-      <pose>13.5 -21 0 0 -0 0</pose>
-    </include>
-    <include>
-      <uri>
-        https://fuel.gazebosim.org/1.0/MovAi/models/shelf
-      </uri>
-      <name>shelf_6</name>
-      <pose>13.5 -15 0 0 -0 0</pose>
-    </include>
-    <include>
-      <uri>
-        https://fuel.gazebosim.org/1.0/MovAi/models/shelf
-      </uri>
-      <name>shelf_7</name>
-      <pose>0.4 -2 0 0 -0 0</pose>
-    </include>
-    <!-- Navigation Challenge section -->
-    <include>
-      <uri>
-        https://fuel.gazebosim.org/1.0/MovAi/models/shelf_big
-      </uri>
-      <name>shelf_big_3</name>
-      <pose>3.5 9.5 0 0 0 1.57</pose>
-    </include>
-    <include>
-      <uri>
-        https://fuel.gazebosim.org/1.0/MovAi/models/shelf_big
-      </uri>
-      <name>shelf_big_4</name>
-      <pose>-1.3 18.5 0 0 0 1.57</pose>
-    </include>
-    <include>
-      <uri>
-        https://fuel.gazebosim.org/1.0/MovAi/models/shelf
-      </uri>
-      <name>shelf_0</name>
-      <pose>-10 21.5 0 0 -0 1.57</pose>
-    </include>
-    <include>
-      <uri>
-        https://fuel.gazebosim.org/1.0/MovAi/models/shelf
-      </uri>
-      <name>shelf_1</name>
-      <pose>-7 23.6 0 0 -0 1.57</pose>
-    </include>
-    <include>
-      <uri>
-        https://fuel.gazebosim.org/1.0/MovAi/models/shelf
-      </uri>
-      <name>shelf_2</name>
-      <pose>-4 21.5 0 0 -0 1.57</pose>
-    </include>
-    <!-- Barriers -->
-    <include>
-      <uri>
-      https://fuel.gazebosim.org/1.0/OpenRobotics/models/Jersey Barrier
-      </uri>
-      <name>barrier_0</name>
-      <pose>-10.4 14.75 0 0 0 1.57</pose>
-    </include>
-    <include>
-      <uri>
-      https://fuel.gazebosim.org/1.0/OpenRobotics/models/Jersey Barrier
-      </uri>
-      <name>barrier_1</name>
-      <pose>-10.4 10.5 0 0 0 1.57</pose>
-    </include>
-    <include>
-      <uri>
-      https://fuel.gazebosim.org/1.0/OpenRobotics/models/Jersey Barrier
-      </uri>
-      <name>barrier_2</name>
-      <pose>-10.4 6.5 0 0 0 1.57</pose>
-    </include>
-    <include>
-      <uri>
-      https://fuel.gazebosim.org/1.0/OpenRobotics/models/Jersey Barrier
-      </uri>
-      <name>barrier_3</name>
-      <pose>-12.85 4.85 0 0 0 0</pose>
-    </include>
-    <!-- Chairs -->
-    <include>
-      <uri>
-        https://fuel.gazebosim.org/1.0/OpenRobotics/models/Chair
-      </uri>
-      <name>chair_0</name>
-      <pose>14.3 -5.5 0 0 -0 3</pose>
-    </include>
-    <include>
-      <uri>
-        https://fuel.gazebosim.org/1.0/OpenRobotics/models/Chair
-      </uri>
-      <name>chair_1</name>
-      <pose>14.3 -4 0 0 -0 -3</pose>
-    </include>
-    <include>
-      <uri>
-        https://fuel.gazebosim.org/1.0/OpenRobotics/models/foldable_chair
-      </uri>
-      <name>fchair_0</name>
-      <pose>-11.5 6.4 0 0 -0 -1.8</pose>
-    </include>
-    <include>
-      <uri>
-        https://fuel.gazebosim.org/1.0/OpenRobotics/models/foldable_chair
-      </uri>
-      <name>fchair1</name>
-      <pose>-14 6.5 0 0 -0 1.9</pose>
-    </include>
-    <!-- Table -->
-    <include>
-      <uri>
-        https://fuel.gazebosim.org/1.0/OpenRobotics/models/CoffeeTable
-      </uri>
-      <name>table0</name>
-      <pose>-12.7 6.5 0 0 0 0</pose>
-    </include>
-    <!-- People -->
-    <include>
-      <uri>
-      https://fuel.gazebosim.org/1.0/OpenRobotics/models/FemaleVisitorSit
-      </uri>
-      <name>Person 0 - Sitting</name>
-      <pose>14.3 -4 0 0 -0 -1.43</pose>
-    </include>
-    <include>
-      <uri>
-      https://fuel.gazebosim.org/1.0/OpenRobotics/models/MaleVisitorOnPhone
-      </uri>
-      <name>Person 1 - Standing</name>
-      <pose>1 -1 0 0 0 1.57</pose>
-    </include>
-    <include>
-      <uri>
-      https://fuel.gazebosim.org/1.0/plateau/models/Casual female
-      </uri>
-      <name>Person 2 - Walking</name>
-      <pose>-12 15 0 0 0 0</pose>
-    </include>
+    <gravity>0 0 -9.8</gravity>
+    <magnetic_field>6e-06 2.3e-05 -4.2e-05</magnetic_field>
+    <atmosphere type='adiabatic'/>
+    <physics name='3ms' type='ode'>
+        <max_step_size>0.003</max_step_size>
+        <real_time_factor>1</real_time_factor>
+    </physics>
+    <scene>
+      <ambient>0.8 0.8 0.8 1</ambient>
+      <background>0.7 0.7 0.7 1</background>
+      <shadows>0</shadows>
+    </scene>
+    <wind/>
+    <spherical_coordinates>
+      <surface_model>EARTH_WGS84</surface_model>
+      <latitude_deg>0</latitude_deg>
+      <longitude_deg>0</longitude_deg>
+      <elevation>0</elevation>
+      <heading_deg>0</heading_deg>
+    </spherical_coordinates>
+    <model name='sim_house'>
+      <pose>1.48679 1.14707 0 0 -0 0</pose>
+      <link name='Wall_0'>
+        <collision name='Wall_0_Collision'>
+          <geometry>
+            <box>
+              <size>2.5 0.15 1</size>
+            </box>
+          </geometry>
+          <pose>0 0 0.5 0 -0 0</pose>
+          <max_contacts>10</max_contacts>
+          <surface>
+            <contact>
+              <ode/>
+            </contact>
+            <bounce/>
+            <friction>
+              <torsional>
+                <ode/>
+              </torsional>
+              <ode/>
+            </friction>
+          </surface>
+        </collision>
+        <visual name='Wall_0_Visual'>
+          <pose>0 0 0.5 0 -0 0</pose>
+          <geometry>
+            <box>
+              <size>2.5 0.15 1</size>
+            </box>
+          </geometry>
+          <material>
+            <script>
+              <uri>file://media/materials/scripts/gazebo.material</uri>
+              <name>Gazebo/Wood</name>
+            </script>
+            <ambient>1 1 1 1</ambient>
+          </material>
+          <meta>
+            <layer>0</layer>
+          </meta>
+        </visual>
+        <pose>-2.70098 -3.18088 0 0 -0 0</pose>
+        <self_collide>0</self_collide>
+        <enable_wind>0</enable_wind>
+        <kinematic>0</kinematic>
+      </link>
+      <link name='Wall_1'>
+        <collision name='Wall_1_Collision'>
+          <geometry>
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